Commit message: P0.6: make the inspection camera reach ROS, and re-spec its mast
The cameras never published because this VM is headless. Without a display Gazebo
cannot initialise OGRE, so no camera sensor is ever created and
libgazebo_ros_camera has nothing to attach to; gzserver.log says exactly that. Both
the inspection webcam and the Astra failed identically, which is the tell that the
fault was in the render engine and not in either sensor. Navigation and the laser
kept working throughout, which is what made the failure easy to misread.

A virtual framebuffer fixes it. xvfb.service (:99, enabled at boot on the sim VM)
now provides the display, and tools/run_neo_workshop.sh resolves one before every
Gazebo launch, falling back to starting its own Xvfb. When it lands on the virtual
framebuffer it also turns RViz off: nobody can see it there and it competes for the
CPU that software rendering needs. Rendering is Mesa llvmpipe — this VM has no GPU —
and the cost is affordable: real-time factor ~1.00 with a camera subscriber against
~1.44 without, at a steady 15.0 Hz.

The mast now models the real 40 x 2 mm aluminium tube the physical build will use:
visual radius 0.010 to 0.020 m, collision 0.012 to 0.022 m, mass 0.35 to 0.62 kg.
Inertia moves to the thick_walled_cylinder_inertia macro, which was already in
inertia.urdf.xacro; the solid-cylinder approximation it replaces understates a
hollow tube. Position, aim and 1280x720 @15 fps / 78 deg HFOV are untouched, and the
optical centre stays at exactly 1.200 m.

Verified: /robot/usb_cam/image_raw steady at ~15.5 Hz with frames that track robot
motion; robot_usb_cam_optical_frame at z = 1.200 m, y = 0; the mast renders as a
40 mm aluminium cylinder; a there-and-back move_base run completes in 42.8 s + 34.9 s
with zero recovery behaviours, against 44.1 s + 38.5 s and zero recoveries before the
mass change. tools/nav_regression_test.py is that check, kept for later regressions.

Note for anything that consumes frames: libgazebo_ros_camera renders only while
subscribed, and the first message after subscribing is the previous session's last
frame with its old timestamp. Hold the subscription and drop the first frame.

Co-Authored-By: Claude Opus 5 <noreply@anthropic.com>

File: rb1_base_common/rb1_base_description/urdf/sensors/usb_cam_webcam.urdf.xacro (robot description, xacro)
@@ -8,13 +8,20 @@
     </joint>
     <link name="${prefix}_mast_link">
+      <!-- Mast modelled as a real 40 x 2 mm aluminium tube (outer diam. 40 mm, 2 mm wall,
+           0.96 m long) because the mount mirrors a planned physical build:
+             cross-section = pi*(0.020^2 - 0.018^2) = 2.388e-4 m^2
+             linear mass   = 2.388e-4 * 2700 kg/m^3 = 0.645 kg/m
+             mast mass     = 0.645 * 0.96          = 0.62 kg
+           Inertia uses the thick-walled tube macro, not the solid-cylinder approximation,
+           which would understate a hollow tube. -->
       <inertial>
-        <mass value="0.35"/>
+        <mass value="0.62"/>
         <origin xyz="0 0 0" rpy="0 0 0"/>
-        <xacro:solid_cylinder_inertia m="0.35" r="0.01" h="0.96"/>
+        <xacro:thick_walled_cylinder_inertia m="0.62" r1="0.018" r2="0.020" h="0.96"/>
       </inertial>
       <visual>
         <origin xyz="0 0 0" rpy="0 0 0"/>
         <geometry>
-          <cylinder radius="0.01" length="0.96"/>
+          <cylinder radius="0.020" length="0.96"/>
         </geometry>
         <material name="usb_cam_mast_aluminum">
@@ -25,5 +32,5 @@
         <origin xyz="0 0 0" rpy="0 0 0"/>
         <geometry>
-          <cylinder radius="0.012" length="0.96"/>
+          <cylinder radius="0.022" length="0.96"/>
         </geometry>
       </collision>
